File: GrasPiB_v1.sch (KiCad schematic (older format))
At the start: 43 parts, among them J1 DB9_Male, J2 Conn_GPIB, J3 JST_PH, J4 JST_PH, J5 3,5mm Pitch, J6 10pin IDC, U1 RPi_GPIO, U2 MAX3232, U3 SN75160BDW, U4 SN75161BDW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

Commit message: Rewire RTS and CTS signals the correct way
Parts:
- C1, C2, C3, C4, C5, C6, C7: symbol Device:C_Small -> GrasPiB_v1-rescue:C_Small-Device
- C8, C9: symbol Device:CP_Small -> GrasPiB_v1-rescue:CP_Small-Device
- D1, D2: symbol Device:LED_Small_ALT -> GrasPiB_v1-rescue:LED_Small_ALT-Device
- D3: symbol Device:D_Schottky_Small_ALT -> GrasPiB_v1-rescue:D_Schottky_Small_ALT-Device
- H1, H2, H3: symbol Mechanical:MountingHole -> GrasPiB_v1-rescue:MountingHole-Mechanical
- J1: symbol Connector:DB9_Male_MountingHoles -> GrasPiB_v1-rescue:DB9_Male_MountingHoles-Connector
- J3: symbol Connector_Generic:Conn_01x02 -> GrasPiB_v1-rescue:Conn_01x02-Connector_Generic
- J4: symbol Connector_Generic:Conn_01x05 -> GrasPiB_v1-rescue:Conn_01x05-Connector_Generic
- J5: symbol Connector:Screw_Terminal_01x02 -> GrasPiB_v1-rescue:Screw_Terminal_01x02-Connector
- J6: symbol Connector_Generic:Conn_02x05_Odd_Even -> GrasPiB_v1-rescue:Conn_02x05_Odd_Even-Connector_Generic
- JP1, JP2, JP4, JP5: symbol Jumper:SolderJumper_2_Open -> GrasPiB_v1-rescue:SolderJumper_2_Open-Jumper
- JP3: symbol Jumper:SolderJumper_3_Bridged12 -> GrasPiB_v1-rescue:SolderJumper_3_Bridged12-Jumper
- JP6: symbol Jumper:SolderJumper_3_Open -> GrasPiB_v1-rescue:SolderJumper_3_Open-Jumper
- JP7: symbol Jumper:Jumper_3_Open -> GrasPiB_v1-rescue:Jumper_3_Open-Jumper
- L1: symbol Device:L_Small -> GrasPiB_v1-rescue:L_Small-Device
- R1, R2, R3, R4, R5: symbol Device:R_Small -> GrasPiB_v1-rescue:R_Small-Device
- RN1, RN2, RN3, RN4: symbol Device:R_Pack04 -> GrasPiB_v1-rescue:R_Pack04-Device
- U2: symbol Interface_UART:MAX3232 -> GrasPiB_v1-rescue:MAX3232-Interface_UART
- U5: symbol Regulator_Switching:LM2576S-5 -> GrasPiB_v1-rescue:LM2576S-5-Regulator_Switching
Connections:
- net UART_CTS: now also U2.9 (R2OUT); no longer U2.10 (T2IN)
- net UART_RTS: now also U2.10 (T2IN); no longer U2.9 (R2OUT)
- net at U2.7 (T2OUT): now also JP5.1 (A); no longer JP4.1 (A)
- net at U2.8 (R2IN): now also JP4.1 (A); no longer JP5.1 (A)
Other:
- moved on the sheet: JP4, JP5
